File: RP2040_Motion_Logger.kicad_sch (KiCad schematic)
At the start: 51 parts, among them J1 Conn_01x02, J3 TC2030-NL, P1 USB_C_Plug_USB2.0, Q1 AO3401A, SW1 RESET, U1 RP2040, U2 TLV62569DBV, U4 MCP73831-2-OT, Y1 12MHZ

Commit message: Added a bootloader button and made some other QOL changes... mostly aesthetic.
Parts:
- removed D3: Green, LED_SMD:LED_0402_1005Metric, symbol Device:LED_Small
- removed R9: 5K, Resistor_SMD:R_0402_1005Metric, symbol Device:R_Small_US
- C18: value 100n -> 4u7; footprint Capacitor_SMD:C_0201_0603Metric -> Capacitor_SMD:C_0402_1005Metric
Connections:
- net USB_D+: now also P1.A6 (D+)
- net USB_D-: now also P1.A7 (D-)
- net GPIO_0 renamed MCU_TX0
- net GPIO_1 renamed MCU_RX0
- net MCU_RX renamed GPIO_ADC3
- net MCU_TX renamed GPIO_ADC2
Other:
- note added: "Battery Charging Circuit"
- note added: "Buck Converter 5 V to 3.3 V max 2 A"
- note added: "Crystal Oscillator"
- note added: "Decoupling Capacitors"
- note added: "ESD Protection"
- note added: "MCU - RP2040"
- note added: "Power Status Led"
- note added: "TC2030 JTAG Connector"
- note added: "USB Type-C"
- moved on the sheet: C1, C2, R1, Y1
