File: sensors_peripherals.kicad_sch (KiCad schematic)
At the start: 17 parts, among them J2 Conn_01x14, J4 Micro_SD_Card_Det1, J5 Conn_01x14, J6 Conn_01x02, U3 W25Q128JVS, U6 ICM-42688-P

Commit message: updated
Other:
- note added: "I2C Pullups"
- company: (none) -> Rishikesh 
- title: (none) -> RP2040 Motion Logger
- moved on the sheet: C20, C21, C22, C23, C26, D4, J2, J4, J5, J6, R10, R15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
